File: KiCad/BikeSensor/BikeSensor.kicad_sch (KiCad schematic)
At the start: 20 parts, among them J1 USB_C_Receptacle_TYPE-C 16PIN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, U1 MDBT50Q-1MV2, U11 TPD4E02B04DQA, U2 LSM6DSV, X1 32.768KHz

Commit message: add: BikeSensor PCB v1 (renamed from RideFormTracker) and the 320X datasheet
The KiCad project is renamed to match what it actually became: not a
RideFormTracker variant but its own 15x33 mm board, with a soft power
latch, BAT_CHECK moved to an analog-capable pin, and an LSM6DSV320X.

Also carries the production files as sent to the fab. Those are
regenerable in principle, but the first article had an open PROG trace -
the charger sat in its shutdown state and neither charged nor lit its
status LED - and being able to compare a board in hand against exactly
what was ordered is worth the few hundred kilobytes.
Parts:
- added TP1, TP2, TP3, TP4, TP5, TP6: TestPoint, TestPoint:TestPoint_Pad_D1.5mm, symbol Connector:TestPoint
- U2: value LSM6DSV -> LSM6DSV320XTR
- U5: now left out of the parts list
Connections:
- net +V_BAT is gone; now on net +3.3V: U5.1 (V)
- net +3.3V: now also TP5.1
- net GND_POWER: now also TP6.1
- net at U1.23 (P0.07): now also TP1.1
- net at U1.25 (P1.08): now also TP2.1
- net at U1.56 (P1.04): now also TP3.1
- net at U1.57 (P1.06): now also TP4.1
