File: KiCad/BikeSensor/Power.kicad_sch (KiCad schematic)
At the start: 17 parts, among them SW2 SW_MEC_5G, U6 BAT, U7 MCP73831-2-MC, U9 TPS7A0233DQNR

Commit message: add: BikeSensor PCB v1 (renamed from RideFormTracker) and the 320X datasheet
The KiCad project is renamed to match what it actually became: not a
RideFormTracker variant but its own 15x33 mm board, with a soft power
latch, BAT_CHECK moved to an analog-capable pin, and an LSM6DSV320X.

Also carries the production files as sent to the fab. Those are
regenerable in principle, but the first article had an open PROG trace -
the charger sat in its shutdown state and neither charged nor lit its
status LED - and being able to compare a board in hand against exactly
what was ordered is worth the few hundred kilobytes.
Parts:
- added H1, H2: (no value), ThroughHole:TH_0.7mm, symbol ThroughHole:TH_0.7
- D2: footprint Diode_SMD:D_0402_1005Metric -> Diode_SMD:D_SOD-323
- U6: now left out of the parts list
- U9: value TPS7A0233DQNR -> TPS7A0233PDQNR
Connections:
- net +V_BAT: now also H1.1
- net GND: now also H2.1

Commit message: add: soft-latch rework, 10M battery divider and a 3D-printed case
Three changes to the enable network, none of which the firmware notices -
the pin assignments are identical, so one image runs on both revisions.

R13 moves to sit in series with SW2. The existing SW_READ divider then
also drops the voltage that reaches LDO_EN, which lands the button path
at 2.97 V instead of 3.95 V. That matters because R12 ties the enable
node straight to P1.11: the old level sat just under the GPIO's ESD
diode and therefore just outside its absolute maximum of VDD + 0.3 V.
Costs nothing - the divider ratio, the SW_READ level and the 9.8 uA
drawn while the button is held are all unchanged.

VBUS reaches the enable node through a 100k/100k divider and D4, so
plugging in USB now starts the board. Previously the button was the only
way in, which was least convenient exactly when the pack was flat. After
a low-battery cutoff a cable now both charges and brings the board up.

With those two, every source that can raise the enable node stays at or
below VDD: 2.25 V from USB, 2.97 V from the button, 3.30 V from the GPIO.

The divider is not there for the LDO's sake - its EN pin is rated to
6.0 V and 5 V direct would be fine. It is there for the GPIO. Dropping
the voltage with a diode's Vf instead cannot work: Vf is a strong
function of current and at I_EN = 10 nA even silicon gives 0.2-0.3 V.
What sets the resistor values is not the ratio but the LDO's 500 kohm
smart enable pulldown, which is engaged at startup and swamps any
divider that is not stiff against it.

The GPIO branch deliberately keeps no diode of its own. Three diodes
would make a symmetric wired-OR, but the GPIO would lose the ability to
pull the enable node DOWN, and today's power-off is an active discharge
through R12 - a one-microsecond time constant that beats any plausible
leakage. Restoring that would need a pulldown, which shortens the
enable node's hold through a reset from ~2 ms to ~100 us and so needs a
capacitor a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
Parts:
- added D4: D, Diode_SMD:D_SOD-323, symbol Device:D
- added R16, R17: 100k, Resistor_SMD:R_0402_1005Metric, symbol Device:R
- R10, R11: value 1M -> 10M
Connections:
- net +5V: now also R16.1
- net GND: now also R15.2, R17.1; no longer R15.1
- net LDO_EN: now also D4.1 (K)
- net SW_READ: now also D2.2 (A), R15.1; no longer R15.2
- net at R13.2, SW2.2 (B), SW2.3 (B): no longer D2.2 (A)
- new net: D4.2 (A), R16.2, R17.2
Other:
- note added: "SoftLatch with LDO_EN"
- note added: "elif GPIO: ON"
- note added: "elif SW: ON"
- note added: "if USB: ON"
- moved on the sheet: D2, R12, R13, R15, SW2
